Commit message: Adjusted the position of the imu

File: opt_ros_indigo_share_husky_description_urdf_husky.urdf.xacro (robot description, xacro)
@@ -89,5 +89,5 @@
     <link name="imu_link"/>
     <joint name="imu_joint" type="fixed">
-      <origin xyz="$(optenv HUSKY_IMU_XYZ 0.19 0 0.149)" rpy="$(optenv HUSKY_IMU_RPY 0 -1.5708 3.1416)" />
+      <origin xyz="$(optenv HUSKY_IMU_XYZ -0.24 0.20 0.18)" rpy="$(optenv HUSKY_IMU_RPY 0 0 3.1416)" />
       <parent link="base_link" />
       <child link="imu_link" />

Commit message: Fixed an error in the frame of the imu

File: opt_ros_indigo_share_husky_description_urdf_husky.urdf.xacro (robot description, xacro)
@@ -89,5 +89,5 @@
     <link name="imu_link"/>
     <joint name="imu_joint" type="fixed">
-      <origin xyz="$(optenv HUSKY_IMU_XYZ -0.24 0.20 0.18)" rpy="$(optenv HUSKY_IMU_RPY 0 0 3.1416)" />
+      <origin xyz="$(optenv HUSKY_IMU_XYZ -0.24 0.20 0.18)" rpy="$(optenv HUSKY_IMU_RPY 3.14159 0 3.14159)" />
       <parent link="base_link" />
       <child link="imu_link" />

Commit message: Add script to create the hardlink

File: opt_ros_indigo_share_husky_description_urdf_husky.urdf.xacro (robot description, xacro)
@@ -95,4 +95,12 @@
     <gazebo reference="imu_link">
     </gazebo>
+    <link name="imu_mit_link"/>
+    <joint name="imu_mit_joint" type="fixed">
+      <origin xyz="$(optenv HUSKY_IMU_MIT_XYZ -0.24 0.20 0.18)" rpy="$(optenv HUSKY_IMU_MIT_RPY 0 0 0)" />
+      <parent link="base_link" />
+      <child link="imu_mit_link" />
+    </joint>
+    <gazebo reference="imu_mit_link">
+    </gazebo>
     <!-- Husky wheel macros -->
     <xacro:husky_wheel wheel_prefix="front_left">

Commit message: Add config for ekf configuration

File: opt_ros_indigo_share_husky_description_urdf_husky.urdf.xacro (robot description, xacro)
@@ -97,5 +97,5 @@
     <link name="imu_mit_link"/>
     <joint name="imu_mit_joint" type="fixed">
-      <origin xyz="$(optenv HUSKY_IMU_MIT_XYZ -0.24 0.20 0.18)" rpy="$(optenv HUSKY_IMU_MIT_RPY 0 0 0)" />
+      <origin xyz="$(optenv HUSKY_IMU_MIT_XYZ -0.24 0.20 0.18)" rpy="$(optenv HUSKY_IMU_MIT_RPY  3.14159 0 -1.5707)" />
       <parent link="base_link" />
       <child link="imu_mit_link" />

Commit message: λ

File: opt_ros_indigo_share_husky_description_urdf_husky.urdf.xacro (robot description, xacro)
@@ -138,6 +138,7 @@
     </xacro:if>
     <xacro:if value="$(arg velodyne_enabled)">
+      <!-- Actual Velodyne -->
       <xacro:HDL-32E parent="top_plate_link" name="velodyne" topic="/velodyne_points">
-          <origin xyz="0 0 0.5" rpy="0 0 0" />
+          <origin xyz="0 0 0" rpy="0 0 0" />
       </xacro:HDL-32E>
     </xacro:if>

Commit message: Correct fix tf error for velodyne.

File: opt_ros_indigo_share_husky_description_urdf_husky.urdf.xacro (robot description, xacro)
@@ -138,6 +138,13 @@
     </xacro:if>
     <xacro:if value="$(arg velodyne_enabled)">
+      <!-- Support, 1.5cm is add to take into account the true high of the user_rail -->
+      <link name="velo_support_base_link"/>
+      <joint name="velo_support_base" type="fixed">
+        <parent link="user_rail_link" />
+        <child link="velo_support_base_link" />
+        <origin xyz="0.023 0 0.15" rpy="0.0 0.0 -1.57" />
+      </joint>
       <!-- Actual Velodyne -->
-      <xacro:HDL-32E parent="top_plate_link" name="velodyne" topic="/velodyne_points">
+      <xacro:HDL-32E parent="velo_support_base_link" name="velodyne" topic="/velodyne_points">
           <origin xyz="0 0 0" rpy="0 0 0" />
       </xacro:HDL-32E>

Commit message: Set husky hostname and changed husky urdf origin.

File: opt_ros_indigo_share_husky_description_urdf_husky.urdf.xacro (robot description, xacro)
@@ -143,5 +143,5 @@
         <parent link="user_rail_link" />
         <child link="velo_support_base_link" />
-        <origin xyz="0.023 0 0.15" rpy="0.0 0.0 -1.57" />
+        <origin xyz="0.023 0 0.15" rpy="0.0 0.0 0.0" />
       </joint>
       <!-- Actual Velodyne -->

Commit message: Changed imu0 and husky urdf.

File: opt_ros_indigo_share_husky_description_urdf_husky.urdf.xacro (robot description, xacro)
@@ -97,5 +97,5 @@
     <link name="imu_mit_link"/>
     <joint name="imu_mit_joint" type="fixed">
-      <origin xyz="$(optenv HUSKY_IMU_MIT_XYZ -0.24 0.20 0.18)" rpy="$(optenv HUSKY_IMU_MIT_RPY  3.14159 0 -1.5707)" />
+      <origin xyz="$(optenv HUSKY_IMU_MIT_XYZ -0.24 0.20 0.18)" rpy="$(optenv HUSKY_IMU_MIT_RPY  0 0 1.5707)" />
       <parent link="base_link" />
       <child link="imu_mit_link" />

Commit message: Updated xsens imu tf.

File: opt_ros_indigo_share_husky_description_urdf_husky.urdf.xacro (robot description, xacro)
@@ -97,5 +97,5 @@
     <link name="imu_mit_link"/>
     <joint name="imu_mit_joint" type="fixed">
-      <origin xyz="$(optenv HUSKY_IMU_MIT_XYZ -0.24 0.20 0.18)" rpy="$(optenv HUSKY_IMU_MIT_RPY  0 0 1.5707)" />
+      <origin xyz="$(optenv HUSKY_IMU_MIT_XYZ -0.24 0.20 0.18)" rpy="$(optenv HUSKY_IMU_MIT_RPY  0 0 3.1416)" />
       <parent link="base_link" />
       <child link="imu_mit_link" />

Commit message: SP Added sick tim-561 support. Velodyne rotated 90 degrees. Changed network interface settings for the new velodyne

File: opt_ros_indigo_share_husky_description_urdf_husky.urdf.xacro (robot description, xacro)
@@ -31,4 +31,5 @@
   <xacro:include filename="$(find ur_description)/urdf/ur5.urdf.xacro" />
   <xacro:include filename="$(find velodyne_description)/urdf/HDL-32E.urdf.xacro" />
+  <xacro:include filename="$(find sick_tim)/urdf/sick_tim.urdf.xacro"/>
   <property name="M_PI" value="3.14159"/>
   <!-- Base Size -->
@@ -147,6 +148,14 @@
       <!-- Actual Velodyne -->
       <xacro:HDL-32E parent="velo_support_base_link" name="velodyne" topic="/velodyne_points">
-          <origin xyz="0 0 0" rpy="0 0 0" />
+          <origin xyz="0 0 0" rpy="0 0 -1.5708" />
       </xacro:HDL-32E>
+    </xacro:if>
+    <xacro:if value="$(arg tim561_enabled)">
+      <xacro:sick_tim551 name="tim561" ros_topic="/scan" />
+      <joint name="tim561_support_base" type="fixed">
+        <parent link="user_rail_link" />
+        <child link="tim561_mount_link" />
+        <origin xyz="0.023 0 0.15" rpy="0.0 0.0 0.0" />
+      </joint>
     </xacro:if>
     <xacro:if value="$(arg kinect_enabled)">
